File: PCB/SPINC AA Charger/SPINC AA Charger.kicad_sch (KiCad schematic)
At the start: 100 parts, among them J1 USB_C_Receptacle_USB2.0, J2 Conn_01x03_Pin, J3 Conn_01x10_Socket, J4 Conn_01x01_Pin, J5 Conn_01x01_Pin, Q1 DMG2301L, Q2 DMHC3025LSD, Q3 DMG2301L, Q4 DMG2301L, Q5 SI2305CDS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

Commit message: LCSC part numbers fixed
- assigned LCSC part numbers properly to the BOM
Parts:
- C1, C3: LCSC C15849 -> C1705
- C10, C13, C14, C16, C18, C19, C21, C22, C24, C26, C27, C28: LCSC (none) -> C1591
- C25, C5: LCSC (none) -> C913904
- C29: LCSC (none) -> C15849
- C30: LCSC C15849 -> C15850
- C7: LCSC C15849 -> C913904
- D2, D4: LCSC (none) -> C26178
- D3: LCSC (none) -> C2928912
- F1: LCSC (none) -> C151162
- J2: LCSC (none) -> C6332196
- L1: LCSC (none) -> C2047110
- Q4: LCSC (none) -> C102619
- Q5: LCSC (none) -> C37577
- R15, R16, R19, R24, R25, R26, R27, R31, R36, R9: LCSC (none) -> C98220
- R18, R23: LCSC (none) -> C99782
- R2: LCSC (none) -> C22548
- R20: LCSC (none) -> C116699
- R21, R22, R28, R29: LCSC (none) -> C105579
- R3, R4: LCSC C114626 -> C105580
- R30: LCSC (none) -> C125923
- R32: LCSC (none) -> C114065
- R33: LCSC (none) -> C14675
- R34: LCSC (none) -> C875831
- R35: LCSC (none) -> C109318
- R37: LCSC (none) -> C105881
- R5: LCSC C114626 -> C14675
- R6: LCSC C114626 -> C245983
- R7, R8: LCSC (none) -> C137753
- U1: LCSC (none) -> C129351
- U3: LCSC C2940197 -> C2940197
